File: PCB/PCB.kicad_pcb (KiCad board)
At the start: 2 copper layers, 3 parts, among them J1 TE1761468-1, SW1 SW_DIP_x01

Commit message: Started pcb
Parts:
- added  : , Connector_PinHeader_2.54mm:PinHeader_1x02_P2.54mm_Horizontal, F.Cu at (94.0, 77.0)
-  : renamed from SW1; value SW_DIP_x01 -> (none)
- moved R1 6.59 mm to (98.0, 77.0)
- moved   2.17 mm to (87.0, 80.0)
Routing:
- net Net-(JP1-Pad1): track 0.00 -> 14.0 mm
- net Net-(J1-Pad1): track 0.00 -> 12.6 mm
- net Net-(J1-Pad4): track 0.00 -> 9.23 mm
- added copper zone on F.Cu, net +12V
- added copper zone on F.Cu, net GND
Other:
- board outline added: 82 x 21 mm

Commit message: PCB Done
Parts:
- removed the   at (94.0, 77.0)
- added  : , MountingHole:MountingHole_6.5mm_Pad, F.Cu at (116.5, 81.0)
- added  : , MountingHole:MountingHole_6.5mm_Pad, F.Cu at (149.5, 81.0)
- added JP1: Jumper_NC_Small, Connector_PinSocket_2.54mm:PinSocket_1x02_P2.54mm_Horizontal, F.Cu at (91.5, 77.0)
- SW1: renamed from  ; value (none) -> SW_DIP_x01
Connections:
- J1 pad 19: +12V -> GND
- J1 pad 46: +12V -> GND
Routing:
- net Net-(J1-Pad1): track 12.6 -> 16.3 mm
- net Net-(JP1-Pad1): track 14.0 -> 16.4 mm
- net GND: vias 0 -> 74
- net +12V: vias 0 -> 80
- added copper zone on B.Cu, net +12V
- added copper zone on B.Cu, net GND

Commit message: Created production files
Routing:
- net Net-(J1-Pad1): track 16.3 -> 22.4 mm
- net Net-(J1-Pad4): track 9.19 -> 14.2 mm
Other:
- board text added: "DPS Board Ethan Cao Rev. 1"
